File: Hardware/GiecoBoard_2021_Rev1/GiecoBoard_2021_Rev1.sch (KiCad schematic (older format))
At the start: 60 parts, among them U1 TM4C129E_Launchpad

Commit message: layout
Parts:
- removed C? (x2): 10uF, symbol Device:C
- removed U?: OKI, symbol MRDT_Devices:OKI
- added C1: 100uF, Capacitor_SMD:C_0603_1608Metric_Pad1.05x0.95mm_HandSolder, symbol Device:C
- added C2: 1000uF, Capacitor_SMD:C_0603_1608Metric_Pad1.05x0.95mm_HandSolder, symbol Device:C
- added D21: GreenLED, LED_SMD:LED_0603_1608Metric_Pad1.05x0.95mm_HandSolder, symbol Device:LED
- added D22: D_Zener, Diode_SMD:D_SOD-323_HandSoldering, symbol Device:D_Zener
- added J10: Test_Point, symbol MRDT_Connectors:Test_Point
- added L1: 100uH, Inductor_SMD:L_0603_1608Metric_Pad1.05x0.95mm_HandSolder, symbol Device:L
- added R21: 330, Resistor_SMD:R_0603_1608Metric_Pad1.05x0.95mm_HandSolder, symbol Device:R
- added U3: LM2576D2TR4-3.3G, symbol MRDT_Devices:LM2576D2TR4-3.3G
- D1, D10, D11, D12, D13, D14, D15, D16, D17, D18, D19, D2, D20, D3, D4, D5, D6, D7, D8, D9: renamed from D?; footprint (none) -> LED_SMD:LED_0603_1608Metric_Pad1.05x0.95mm_HandSolder
- J1, J11, J2, J3, J4, J5, J6, J7, J8, J9: renamed from J?; footprint (none) -> Button_Switch_SMD:SW_DIP_SPSTx02_Slide_6.7x6.64mm_W6.73mm_P2.54mm_LowProfile_JPin
- R1, R10, R11, R12, R13, R14, R15, R16, R17, R18, R19, R2, R20, R3, R4, R5, R6, R7, R8, R9: renamed from R?; footprint (none) -> Resistor_SMD:R_0603_1608Metric_Pad1.05x0.95mm_HandSolder
- U1: footprint MRDT_Shields:TM4C129E_Launchpad_FULL_SMD_BOTTOM -> MRDT_Shields:TM4C129E_Launchpad_FULL_THT_TOP
- U1: renamed from U?; footprint (none) -> MRDT_Shields:TM4C129E_Launchpad_FULL_THT_TOP
Connections:
- wire segments 146 -> 198
Other:
- note added: "3.3V Buck Conv."
- note removed: "12v to 3.3v oki"

Commit message: layout
Connections:
- net labels added: ON_LED_NavigationalControl, REC_LED_NavigationalControl
- net labels removed: ON_LED_NacigationalControl, REC_LED_NacigationalControl
Changed lines of the file:
@@
 ON_LED_DriveCommand
 Text GLabel 6350 2950 0    39   Input ~ 0
-ON_LED_NacigationalControl
+ON_LED_NavigationalControl
 Text GLabel 6350 3350 0    39   Input ~ 0
 ON_LED_12VDistribution
@@
 REC_LED_DriveCommand
 Text GLabel 8400 2950 0    39   Input ~ 0
-REC_LED_NacigationalControl
+REC_LED_NavigationalControl
 Text GLabel 8400 3350 0    39   Input ~ 0
 REC_LED_12VDistribution
@@
 ON_LED_DriveCommand
 Text GLabel 1450 2750 2    39   Output ~ 0
-ON_LED_NacigationalControl
+ON_LED_NavigationalControl
 Text GLabel 1450 2850 2    39   Output ~ 0
 ON_LED_12VDistribution
@@
 REC_LED_DriveCommand
 Text GLabel 3500 2750 0    39   Output ~ 0
-REC_LED_NacigationalControl
+REC_LED_NavigationalControl
 Text GLabel 3500 2850 0    39   Output ~ 0
 REC_LED_12VDistribution

Commit message: schematic
Parts:
- J1, J2, J3, J4, J5, J6, J7, J8, J9: footprint Button_Switch_SMD:SW_DIP_SPSTx02_Slide_6.7x6.64mm_W6.73mm_P2.54mm_LowProfile_JPin -> Button_Switch_THT:SW_PUSH-12mm
Connections:
- net labels added: ON_LED_ScienceActuation, REC_LED_ScienceActuation
- net labels removed: ON_LED_SciencnActuation, REC_LED_SciencnActuation
- wire segments 198 -> 204

Commit message: changeLED resistors value
Parts:
- removed D1, D11, D13, D15, D17, D19, D3, D5, D7, D9: GreenLED, LED_SMD:LED_0603_1608Metric_Pad1.05x0.95mm_HandSolder, symbol Device:LED
- removed D10, D12, D14, D16, D18, D2, D20, D4, D6, D8: BlueLED, LED_SMD:LED_0603_1608Metric_Pad1.05x0.95mm_HandSolder, symbol Device:LED
- removed R1, R10, R11, R12, R13, R14, R15, R16, R17, R18, R19, R2, R20, R3, R4, R5, R6, R7, R8, R9: 500, Resistor_SMD:R_0603_1608Metric_Pad1.05x0.95mm_HandSolder, symbol Device:R
- added D? (x20): LED, symbol Device:LED
- added R? (x20): 330, symbol Device:R
- D21: value GreenLED -> LED
Other:
- note added: "Green"

Commit message: Annotate and colored LEDs
Parts:
- gave numbers to parts that had none: 40
Other:
- note added: "Yellow"

Commit message: 1st_BoardReviewChange
Parts:
- removed D11, D13, D15, D17, D19, D3, D5, D7, D9: LED, symbol Device:LED
- removed J11: Conn_02x02_Top_Bottom, Button_Switch_SMD:SW_DIP_SPSTx02_Slide_6.7x6.64mm_W6.73mm_P2.54mm_LowProfile_JPin, symbol Connector_Generic:Conn_02x02_Top_Bottom
- removed J2, J3, J4, J5, J6, J7, J8, J9: Conn_02x02_Top_Bottom, Button_Switch_THT:SW_PUSH-12mm, symbol Connector_Generic:Conn_02x02_Top_Bottom
- removed R11, R13, R15, R17, R19, R3, R5, R7, R9: 330, symbol Device:R
- added Conn? (x2): AndersonPP, symbol MRDT_Connectors:AndersonPP
- added D? (x9): LED, LED_SMD:LED_0603_1608Metric_Pad1.05x0.95mm_HandSolder, symbol Device:LED
- added J? (x9): Conn_02x02_Top_Bottom, Button_Switch_THT:SW_PUSH-12mm, symbol Connector_Generic:Conn_02x02_Top_Bottom
- added R? (x9): 330, Resistor_SMD:R_0603_1608Metric_Pad1.05x0.95mm_HandSolder, symbol Device:R
- D1, D10, D12, D14, D16, D18, D2, D20, D4, D6, D8: footprint (none) -> LED_SMD:LED_0603_1608Metric_Pad1.05x0.95mm_HandSolder
- R1, R10, R12, R14, R16, R18, R2, R20, R4, R6, R8: footprint (none) -> Resistor_SMD:R_0603_1608Metric_Pad1.05x0.95mm_HandSolder
Connections:
- net labels removed: ON_LED_12VDistribution, ON_LED_ArmArticulation, ON_LED_BatteryManagement, ON_LED_DriveCommand, ON_LED_Gimbal, ON_LED_Multimedia, ON_LED_NavigationalControl, ON_LED_PackVoltageDistribution, ON_LED_ScienceActuation, ON_LED_ScienceSensor
- wire segments 204 -> 213
Other:
- note added: "12V Anderson"
- note added: "Blue"
- note added: "SendSigBottoms \nwith ON/OFF LED"
- note removed: "ON/OFF LED"
- note removed: "SendSigBottoms"
- note removed: "Yellow"
