File: Hardware/GiecoBoard_2021_Rev1/GiecoBoard_2021_Rev1.sch (KiCad schematic (older format))
At the start: 61 parts, among them J1 Conn_02x02_Top_Bottom, J10 Test_Point, U1 TM4C129E_Launchpad, U3 LM2576D2TR4-3.3G

Commit message: layout_no wiring
Parts:
- removed Conn?: AndersonPP, symbol MRDT_Connectors:AndersonPP
- removed D22: D_Zener, Diode_SMD:D_SOD-323_HandSoldering, symbol Device:D_Zener
- removed U3: LM2576D2TR4-3.3G, symbol MRDT_Devices:LM2576D2TR4-3.3G
- added unit 2 of Conn1
- added D22: D_Schottky, Diode_SMD:D_SOD-323_HandSoldering, symbol Device:D_Schottky
- added U2: LM2576D2TR4, MRDT_Devices:LM2576, symbol MRDT_Devices:LM2576D2TR4
- Conn1: renamed from Conn?; footprint (none) -> MRDT_Connectors:Anderson_2_Horizontal_Side_by_Side
- J10: footprint (none) -> TestPoint:TestPoint_THTPad_1.0x1.0mm_Drill0.5mm
- gave numbers to parts that had none: 27
Connections:
- net labels removed: +12V
- wire segments 213 -> 265
- no-connect marks 0 -> 54
Other:
- note added: "& 12V Anderson"
- note removed: "12V Anderson"

Commit message: fliped tiva_pin on layout
Changed lines of the file:
@@
 Wire Wire Line
 	3950 900  3950 1200
-Text GLabel 1450 1400 2    39   Output ~ 0
+Text GLabel 1450 1500 2    39   Output ~ 0
 REC_LED_ArmArticulation
-Text GLabel 1450 1700 2    39   Output ~ 0
+Text GLabel 1450 1800 2    39   Output ~ 0
 REC_LED_ScienceSensor
 Text GLabel 1450 2100 2    39   Output ~ 0
@@
 Text GLabel 4000 1400 2    39   Output ~ 0
 REC_LED_DriveCommand
-Text GLabel 1450 2850 2    39   Output ~ 0
+Text GLabel 1450 2950 2    39   Output ~ 0
 REC_LED_NavigationalControl
-Text GLabel 1450 3250 2    39   Output ~ 0
+Text GLabel 1450 3350 2    39   Output ~ 0
 REC_LED_12VDistribution
-Text GLabel 4000 3250 2    39   Output ~ 0
+Text GLabel 4000 3350 2    39   Output ~ 0
 REC_LED_BatteryManagement
-Text GLabel 4000 2750 2    39   Output ~ 0
+Text GLabel 4000 2850 2    39   Output ~ 0
 REC_LED_PackVoltageDistribution
 Text GLabel 4000 2100 2    39   Output ~ 0
@@
 Wire Wire Line
 	4000 2100 3950 2100
-Text GLabel 1450 1500 2    39   Input ~ 0
+Text GLabel 1450 1400 2    39   Input ~ 0
 Send_ArmArticulation
-Text GLabel 1450 1800 2    39   Input ~ 0
+Text GLabel 1450 1700 2    39   Input ~ 0
 Send_ScienceSensor
 Text GLabel 1450 2000 2    39   Input ~ 0
@@
 Text GLabel 4000 1300 2    39   Input ~ 0
 Send_DriveCommand
-Text GLabel 1450 2950 2    39   Input ~ 0
+Text GLabel 1450 2850 2    39   Input ~ 0
 Send_NavigationalControl
-Text GLabel 1450 3350 2    39   Input ~ 0
+Text GLabel 1450 3250 2    39   Input ~ 0
 Send_12VDistribution
-Text GLabel 4000 3350 2    39   Input ~ 0
+Text GLabel 4000 3250 2    39   Input ~ 0
 Send_BatteryManagement
-Text GLabel 4000 2850 2    39   Input ~ 0
+Text GLabel 4000 2750 2    39   Input ~ 0
 Send_PackVoltageDistribution
 Text GLabel 4000 2000 2    39   Input ~ 0

Commit message: wiring on layout
Connections:
- wire segments 265 -> 267
Changed lines of the file:
@@
 L power:+3.3V #PWR012
 U 1 1 5F686880
-P 500 2450
-F 0 "#PWR012" H 500 2300 50  0001 C CNN
-F 1 "+3.3V" H 515 2623 50  0000 C CNN
-F 2 "" H 500 2450 50  0001 C CNN
-F 3 "" H 500 2450 50  0001 C CNN
-	1    500  2450
+P 450 2500
+F 0 "#PWR012" H 450 2350 50  0001 C CNN
+F 1 "+3.3V" H 465 2673 50  0000 C CNN
+F 2 "" H 450 2500 50  0001 C CNN
+F 3 "" H 450 2500 50  0001 C CNN
+	1    450  2500
 	1    0    0    -1
 $EndComp
@@
 L power:+3.3V #PWR02
 U 1 1 5F6888BC
-P 500 1100
-F 0 "#PWR02" H 500 950 50  0001 C CNN
-F 1 "+3.3V" H 515 1273 50  0000 C CNN
-F 2 "" H 500 1100 50  0001 C CNN
-F 3 "" H 500 1100 50  0001 C CNN
-	1    500  1100
-	1    0    0    -1
-$EndComp
-Wire Wire Line
-	500  1200 500  1100
-Wire Wire Line
-	500  2550 500  2450
+P 450 1150
+F 0 "#PWR02" H 450 1000 50  0001 C CNN
+F 1 "+3.3V" H 465 1323 50  0000 C CNN
+F 2 "" H 450 1150 50  0001 C CNN
+F 3 "" H 450 1150 50  0001 C CNN
+	1    450  1150
+	1    0    0    -1
+$EndComp
 $Comp
 L power:GND #PWR01
@@
 	0    1    1    0
 $EndComp
+Wire Wire Line
+	500  1200 450  1200
+Wire Wire Line
+	450  1200 450  1150
+Wire Wire Line
+	500  2550 450  2550
+Wire Wire Line
+	450  2550 450  2500
 $EndSCHEMATC

Commit message: fix 3.3v buck
Parts:
- U2: value LM2576D2TR4 -> LM2576SX-3.3
Changed lines of the file:
@@
 P 1800 7350
 F 0 "U2" H 1800 7775 50  0000 C CNN
-F 1 "LM2576D2TR4" H 1800 7684 50  0000 C CNN
+F 1 "LM2576SX-3.3" H 1800 7684 50  0000 C CNN
 F 2 "MRDT_Devices:LM2576" H 1800 7800 50  0001 C CNN
 F 3 "https://www.mouser.com/datasheet/2/308/LM2576_D-1810688.pdf" H 1800 7800 50  0001 C CNN

Commit message: Layout review update
Parts:
- Conn1: footprint MRDT_Connectors:Anderson_2_Horizontal_Side_by_Side -> MRDT_Connectors:Anderson_2_Vertical_Sidy_by_Side
- D22: value D_Schottky -> 1n5582; footprint Diode_SMD:D_SOD-323_HandSoldering -> Diode_THT:D_DO-201AD_P15.24mm_Horizontal
Changed lines of the file:
@@
 F 0 "Conn1" H 2106 6687 60  0000 C CNN
 F 1 "AndersonPP" H 2106 6581 60  0000 C CNN
-F 2 "MRDT_Connectors:Anderson_2_Horizontal_Side_by_Side" H 1750 5750 60  0001 C CNN
+F 2 "MRDT_Connectors:Anderson_2_Vertical_Sidy_by_Side" H 1750 5750 60  0001 C CNN
 F 3 "" H 1750 5750 60  0001 C CNN
 	1    1900 6300
@@
 F 0 "Conn1" H 2106 7187 60  0000 C CNN
 F 1 "AndersonPP" H 2106 7081 60  0000 C CNN
-F 2 "MRDT_Connectors:Anderson_2_Horizontal_Side_by_Side" H 1750 6250 60  0001 C CNN
+F 2 "MRDT_Connectors:Anderson_2_Vertical_Sidy_by_Side" H 1750 6250 60  0001 C CNN
 F 3 "" H 1750 6250 60  0001 C CNN
 	2    1900 6800
@@
 P 2550 7500
 F 0 "D22" H 2550 7716 50  0000 C CNN
-F 1 "D_Schottky" H 2550 7625 50  0000 C CNN
-F 2 "Diode_SMD:D_SOD-323_HandSoldering" H 2550 7500 50  0001 C CNN
+F 1 "1n5582" H 2550 7625 50  0000 C CNN
+F 2 "Diode_THT:D_DO-201AD_P15.24mm_Horizontal" H 2550 7500 50  0001 C CNN
 F 3 "~" H 2550 7500 50  0001 C CNN
 	1    2550 7500

Commit message: change TIVA footprint
Parts:
- U1: footprint MRDT_Shields:TM4C129E_Launchpad_FULL_THT_TOP -> MRDT_Shields:TM4C129E_Launchpad_FULL_THT_BOTTOM
Changed lines of the file:
@@
 F 0 "U1" H 3300 3350 60  0000 L CNN
 F 1 "TM4C129E_Launchpad" H 2150 4650 60  0000 L CNN
-F 2 "MRDT_Shields:TM4C129E_Launchpad_FULL_THT_TOP" H 3250 3500 60  0001 C CNN
+F 2 "MRDT_Shields:TM4C129E_Launchpad_FULL_THT_BOTTOM" H 3250 3500 60  0001 C CNN
 F 3 "" H 3250 3500 60  0001 C CNN
 	7    3250 3500
@@
 F 0 "U1" H 3850 4650 60  0000 C CNN
 F 1 "TM4C129E_Launchpad" H 3400 3250 60  0001 C CNN
-F 2 "MRDT_Shields:TM4C129E_Launchpad_FULL_THT_TOP" H 3750 3500 60  0001 C CNN
+F 2 "MRDT_Shields:TM4C129E_Launchpad_FULL_THT_BOTTOM" H 3750 3500 60  0001 C CNN
 F 3 "" H 3750 3500 60  0001 C CNN
 	8    3750 3500
@@
 F 0 "U1" H 750 3350 60  0000 L CNN
 F 1 "TM4C129E_Launchpad" H 1100 4000 60  0001 L CNN
-F 2 "MRDT_Shields:TM4C129E_Launchpad_FULL_THT_TOP" H 700 3500 60  0001 C CNN
+F 2 "MRDT_Shields:TM4C129E_Launchpad_FULL_THT_BOTTOM" H 700 3500 60  0001 C CNN
 F 3 "" H 700 3500 60  0001 C CNN
 	5    700  3500
@@
 F 0 "U1" H 1300 4650 60  0000 C CNN
 F 1 "TM4C129E_Launchpad" H 1600 1900 60  0001 C CNN
-F 2 "MRDT_Shields:TM4C129E_Launchpad_FULL_THT_TOP" H 1200 3500 60  0001 C CNN
+F 2 "MRDT_Shields:TM4C129E_Launchpad_FULL_THT_BOTTOM" H 1200 3500 60  0001 C CNN
 F 3 "" H 1200 3500 60  0001 C CNN
 	6    1200 3500
@@
 F 0 "U1" H 750 2000 60  0000 L CNN
 F 1 "TM4C129E_Launchpad" H 1500 3250 60  0001 L CNN
-F 2 "MRDT_Shields:TM4C129E_Launchpad_FULL_THT_TOP" H 700 2150 60  0001 C CNN
+F 2 "MRDT_Shields:TM4C129E_Launchpad_FULL_THT_BOTTOM" H 700 2150 60  0001 C CNN
 F 3 "" H 700 2150 60  0001 C CNN
 	1    700  2150
@@
 F 0 "U1" H 1350 3300 60  0000 C CNN
 F 1 "TM4C129E_Launchpad" H 1250 2550 60  0001 C CNN
-F 2 "MRDT_Shields:TM4C129E_Launchpad_FULL_THT_TOP" H 1200 2150 60  0001 C CNN
+F 2 "MRDT_Shields:TM4C129E_Launchpad_FULL_THT_BOTTOM" H 1200 2150 60  0001 C CNN
 F 3 "" H 1200 2150 60  0001 C CNN
 	2    1200 2150
@@
 F 0 "U1" H 3300 2000 60  0000 L CNN
 F 1 "TM4C129E_Launchpad" H 3650 2700 60  0001 L CNN
-F 2 "MRDT_Shields:TM4C129E_Launchpad_FULL_THT_TOP" H 3250 2150 60  0001 C CNN
+F 2 "MRDT_Shields:TM4C129E_Launchpad_FULL_THT_BOTTOM" H 3250 2150 60  0001 C CNN
 F 3 "" H 3250 2150 60  0001 C CNN
 	3    3250 2150
@@
 F 0 "U1" H 3900 3300 60  0000 C CNN
 F 1 "TM4C129E_Launchpad" H 3450 3250 60  0001 C CNN
-F 2 "MRDT_Shields:TM4C129E_Launchpad_FULL_THT_TOP" H 3750 2150 60  0001 C CNN
+F 2 "MRDT_Shields:TM4C129E_Launchpad_FULL_THT_BOTTOM" H 3750 2150 60  0001 C CNN
 F 3 "" H 3750 2150 60  0001 C CNN
 	4    3750 2150

Commit message: Post CDR update
Parts:
- removed D2: LED, LED_SMD:LED_0603_1608Metric_Pad1.05x0.95mm_HandSolder, symbol Device:LED
- removed D22: 1n5582, Diode_THT:D_DO-201AD_P15.24mm_Horizontal, symbol Device:D_Schottky
- removed J10: Test_Point, TestPoint:TestPoint_THTPad_1.0x1.0mm_Drill0.5mm, symbol MRDT_Connectors:Test_Point
- removed L1: 100uH, Inductor_SMD:L_0603_1608Metric_Pad1.05x0.95mm_HandSolder, symbol Device:L
- removed U2: LM2576SX-3.3, MRDT_Devices:LM2576, symbol MRDT_Devices:LM2576D2TR4
- added D1: Green, LED_SMD:LED_0603_1608Metric_Pad1.05x0.95mm_HandSolder, symbol Device:LED
- added U2: OKI, MRDT_Devices:OKI_Horizontal, symbol MRDT_Devices:OKI
- C1: value 100uF -> 10uF
- C2: value 1000uF -> 10uF
- D10, D12, D15, D17, D18, D19, D20, D5, D7: value LED -> Blue
- D11, D13, D14, D16, D21, D3, D4, D6, D8, D9: value LED -> Green
- D2: renamed from D1; value LED -> Blue
- renumbered J11 to J10, R2 to R1, R7 to R10, R14 to R11, R9 to R12, R16 to R13, R18 to R14, R11 to R15, R20 to R16, R13 to R17, R15 to R18, R17 to R19, R1 to R2, R19 to R20, R4 to R3, R6 to R4, R3 to R5, R8 to R6, R5 to R7, R10 to R8, R12 to R9
Connections:
- wire segments 267 -> 252
Other:
- note removed: "Blue"
- note removed: "Green"
